File: electronics/buttons.sch (KiCad schematic (older format))
At the start: 8 parts, among them J1 Conn_01x02, J2 Conn_01x02, J3 Conn_01x02, J4 Conn_01x02, SW1 SW_Push, SW2 SW_Push, SW3 SW_Push, SW4 SW_Push

Commit message: Schematic of ring for lambda/4
Parts:
- J1, J2, J3, J4: footprint my_footprints:SMD2pin -> Pin_Headers.pretty:Pin_Header_Straight_1x02_Pitch2.54mm
Changed lines of the file:
@@
 LIBS:contrib
 LIBS:valves
+LIBS:buttons-cache
 EELAYER 25 0
 EELAYER END
@@
 F 0 "J1" H 4100 1950 50  0000 C CNN
 F 1 "Conn_01x02" H 4100 1650 50  0000 C CNN
-F 2 "my_footprints:SMD2pin" H 4100 1850 50  0001 C CNN
+F 2 "Pin_Headers.pretty:Pin_Header_Straight_1x02_Pitch2.54mm" H 4100 1850 50  0001 C CNN
 F 3 "" H 4100 1850 50  0001 C CNN
 	1    4100 1850
@@
 F 0 "J2" H 4100 2400 50  0000 C CNN
 F 1 "Conn_01x02" H 4100 2100 50  0000 C CNN
-F 2 "my_footprints:SMD2pin" H 4100 2300 50  0001 C CNN
+F 2 "Pin_Headers.pretty:Pin_Header_Straight_1x02_Pitch2.54mm" H 4100 2300 50  0001 C CNN
 F 3 "" H 4100 2300 50  0001 C CNN
 	1    4100 2300
@@
 F 0 "J3" H 4100 2850 50  0000 C CNN
 F 1 "Conn_01x02" H 4100 2550 50  0000 C CNN
-F 2 "my_footprints:SMD2pin" H 4100 2750 50  0001 C CNN
+F 2 "Pin_Headers.pretty:Pin_Header_Straight_1x02_Pitch2.54mm" H 4100 2750 50  0001 C CNN
 F 3 "" H 4100 2750 50  0001 C CNN
 	1    4100 2750
@@
 F 0 "J4" H 4100 3300 50  0000 C CNN
 F 1 "Conn_01x02" H 4100 3000 50  0000 C CNN
-F 2 "my_footprints:SMD2pin" H 4100 3200 50  0001 C CNN
+F 2 "Pin_Headers.pretty:Pin_Header_Straight_1x02_Pitch2.54mm" H 4100 3200 50  0001 C CNN
 F 3 "" H 4100 3200 50  0001 C CNN
 	1    4100 3200
